Commit message: Update models

File: hector_quadrotor_description/urdf/quadrotor_base_plus.urdf.xacro (robot description, xacro)
@@ -14,5 +14,5 @@
         <origin xyz="0 0 0" rpy="0 0 0" />
         <geometry>
-          <mesh filename="package://hector_quadrotor_description/meshes/quadrotor/quadrotor_CAD2.dae"/>
+          <mesh filename="package://hector_quadrotor_description/meshes/quadrotor/quadrotor_CAD2_visuals.dae"/>
         </geometry>
       </visual>
@@ -20,5 +20,5 @@
         <origin xyz="0 0 0" rpy="0 0 0" />
         <geometry>
-          <mesh filename="package://hector_quadrotor_description/meshes/quadrotor/quadrotor_CAD2.stl"/>
+          <mesh filename="package://hector_quadrotor_description/meshes/quadrotor/quadrotor_CAD2_collision.stl"/>
         </geometry>
       </collision>

File: hector_quadrotor_description/urdf/quadrotor_plus.urdf.xacro (robot description, xacro)
@@ -7,7 +7,7 @@
     <xacro:quadrotor_base_macro />
     <!-- Forward facing camera -->
-    <xacro:include filename="$(find hector_sensors_description)/urdf/generic_camera.urdf.xacro" />
-    <xacro:generic_camera name="front_cam" parent="base_link" ros_topic="camera/image" cam_info_topic="camera/camera_info" update_rate="10" res_x="640" res_y="480" image_format="R8G8B8" hfov="90">
-      <origin xyz="-0.05 0.0 -0.06" rpy="0 0.78539 0"/>  <!-- PI / 4 = 0.78539 = 45deg -->
+    <xacro:include filename="$(find hector_sensors_description)/urdf/generic_camera_plus.urdf.xacro" />
+    <xacro:generic_camera name="front_cam" parent="base_link" ros_topic="camera/image" cam_info_topic="camera/camera_info" update_rate="10" res_x="960" res_y="720" image_format="R8G8B8" hfov="90">
+      <origin xyz="0.05 0.0 -0.06" rpy="0 0.5890 0"/>  <!-- PI / 4 = 0.78539 = 45deg -->
     </xacro:generic_camera>
 </robot>

Commit message: Comply with rules for links

File: hector_quadrotor_description/urdf/quadrotor_base_plus.urdf.xacro (robot description, xacro)
@@ -24,8 +24,72 @@
       </collision>
     </link>
-    <!-- Sonar height sensor -->
-    <xacro:sonar_sensor name="sonar" parent="base_link" ros_topic="sonar_height" update_rate="10" min_range="0.03" max_range="3.0" field_of_view="${40*pi/180}" ray_count="3">
-      <origin xyz="-0.16 0.0 -0.012" rpy="0 ${90*pi/180} 0"/>
-    </xacro:sonar_sensor>
+    <!-- Fixed Joint from Core to Rod -->
+    <joint name="core_to_rod" type="fixed">
+        <parent link="base_link"/>
+        <child link="rod_link"/>
+        <origin xyz="0.05 0 0" rpy="0 0 0"/> <!-- Adjust offset as needed -->
+    </joint>
+    <!-- Rod Link -->
+    <link name="rod_link">
+        <visual>
+        <geometry>
+            <cylinder length="0.06" radius="0.005"/> <!-- Thin rod -->
+        </geometry>
+        <material name="black"/>
+        </visual>
+        <inertial>
+            <mass value="0.01" />
+            <origin xyz="0 0 0" />
+            <inertia ixx="0.0" ixy="0.0" ixz="0.0" iyy="0.0" iyz="0.0" izz="0.0" />
+      </inertial>
+    </link>
+    <!-- Fixed Joint from Rod to Camera -->
+    <joint name="rod_to_camera" type="fixed">
+        <parent link="rod_link"/>
+        <child link="camera_link"/>
+        <origin xyz="0 0 -0.05" rpy="0 0 0"/>
+    </joint>
+    <!-- Camera Link -->
+    <link name="camera_link">
+        <inertial>
+            <mass value="0.01" />
+            <origin xyz="0 0 0" />
+            <inertia ixx="0.0" ixy="0.0" ixz="0.0" iyy="0.0" iyz="0.0" izz="0.0" />
+      </inertial>
+    </link>
+        <!-- Fixed Joint from Core to Rod -->
+    <joint name="core_to_depth_camera_rod" type="fixed">
+        <parent link="base_link"/>
+        <child link="depth_camera_rod_link"/>
+        <origin xyz="0 0 0" rpy="0 0 0"/>
+    </joint>
+        <!-- Rod Link -->
+    <link name="depth_camera_rod_link">
+        <visual>
+        <geometry>
+            <cylinder length="0.03" radius="0.005"/> <!-- Thin rod -->
+        </geometry>
+        <material name="black"/>
+        </visual>
+        <inertial>
+            <mass value="0.01" />
+            <origin xyz="0 0 0" />
+            <inertia ixx="0.0" ixy="0.0" ixz="0.0" iyy="0.0" iyz="0.0" izz="0.0" />
+      </inertial>
+    </link>
+    <!-- Fixed Joint from Rod to Camera -->
+    <joint name="rod_to_depth_camera" type="fixed">
+        <parent link="depth_camera_rod_link"/>
+        <child link="depth_camera_link"/>
+        <origin xyz="0 0 -0.03" rpy="0 0 0"/>
+    </joint>
+    <!-- Camera Link -->
+    <link name="depth_camera_link">
+        <inertial>
+            <mass value="0.01" />
+            <origin xyz="0 0 0" />
+            <inertia ixx="0.0" ixy="0.0" ixz="0.0" iyy="0.0" iyz="0.0" izz="0.0" />
+      </inertial>
+    </link>
   </xacro:macro>
 </robot>

File: hector_quadrotor_description/urdf/quadrotor_plus.urdf.xacro (robot description, xacro)
@@ -8,8 +8,26 @@
     <!-- Forward facing camera -->
     <xacro:include filename="$(find hector_sensors_description)/urdf/generic_camera_plus.urdf.xacro" />
-    <xacro:generic_camera name="front_cam" parent="base_link" ros_topic="camera/image" cam_info_topic="camera/camera_info" update_rate="10" res_x="1280" res_y="960" image_format="R8G8B8" hfov="90">
-      <origin xyz="0.05 0.0 -0.06" rpy="0 0.5890 0"/>  <!-- PI / 4 = 0.78539 = 45deg -->
+    <xacro:generic_camera name="front_cam" parent="camera_link" ros_topic="camera/image" cam_info_topic="camera/camera_info" update_rate="10" res_x="1280" res_y="960" image_format="R8G8B8" hfov="90">
+      <origin xyz="0.0 0.0 0.0" rpy="0 0.5890 0"/>  <!-- PI / 4 = 0.78539 = 45deg -->
     </xacro:generic_camera>
-    <gazebo reference="base_link">
+    <joint name="depth_camera_joint" type="fixed">
+        <origin xyz="0 0 0" rpy="0 0 0"/>
+        <parent link="depth_camera_link"/>
+        <child link="depth_camera_optical_link"/>
+    </joint>
+    <link name="depth_camera_optical_link">
+        <inertial>
+            <mass value="0.01" />
+            <origin xyz="0 0 0" rpy="0 0 0" />
+            <inertia ixx="0" ixy="0" ixz="0" iyy="0" iyz="0" izz="0" />
+        </inertial>
+        <visual>
+            <origin xyz="0 0 0" rpy="0 1.571 0" />
+            <geometry>
+            <mesh filename="package://hector_sensors_description/meshes/hokuyo_utm30lx/hokuyo_utm30lx.dae"/>
+        </geometry>
+        </visual>
+    </link>
+    <gazebo reference="depth_camera_optical_link">
         <!-- Combined Depth and RGB Camera Sensor -->
         <sensor type="depth" name="combined_camera">

Commit message: Adjust links

File: hector_quadrotor_description/urdf/quadrotor_base_plus.urdf.xacro (robot description, xacro)
@@ -34,5 +34,5 @@
         <visual>
         <geometry>
-            <cylinder length="0.06" radius="0.005"/> <!-- Thin rod -->
+            <cylinder length="0.05" radius="0.005"/> <!-- Thin rod -->
         </geometry>
         <material name="black"/>
@@ -48,5 +48,5 @@
         <parent link="rod_link"/>
         <child link="camera_link"/>
-        <origin xyz="0 0 -0.05" rpy="0 0 0"/>
+        <origin xyz="0 0 -0.04" rpy="0 0 0"/>
     </joint>
     <!-- Camera Link -->
@@ -68,5 +68,5 @@
         <visual>
         <geometry>
-            <cylinder length="0.03" radius="0.005"/> <!-- Thin rod -->
+            <cylinder length="0.02" radius="0.005"/> <!-- Thin rod -->
         </geometry>
         <material name="black"/>
@@ -82,5 +82,5 @@
         <parent link="depth_camera_rod_link"/>
         <child link="depth_camera_link"/>
-        <origin xyz="0 0 -0.03" rpy="0 0 0"/>
+        <origin xyz="0 0 -0.02" rpy="0 0 0"/>
     </joint>
     <!-- Camera Link -->
