Commit message: Fix camera angle to 45deg

File: hector_quadrotor_description/urdf/quadrotor_plus.urdf.xacro (robot description, xacro)
@@ -9,5 +9,5 @@
     <xacro:include filename="$(find hector_sensors_description)/urdf/generic_camera.urdf.xacro" />
     <xacro:generic_camera name="front_cam" parent="base_link" ros_topic="camera/image" cam_info_topic="camera/camera_info" update_rate="10" res_x="320" res_y="240" image_format="R8G8B8" hfov="90">
-      <origin xyz="-0.05 0.0 -0.06" rpy="0 1.5707 0"/>  <!-- PI / 2 = 1.5707 -->
+      <origin xyz="-0.05 0.0 -0.06" rpy="0 0.78539 0"/>  <!-- PI / 4 = 0.78539 = 45deg -->
     </xacro:generic_camera>
 </robot>

Commit message: Fix camera orientation

File: hector_quadrotor_description/urdf/quadrotor_plus.urdf.xacro (robot description, xacro)
@@ -12,5 +12,5 @@
     </xacro:generic_camera>
     <joint name="depth_camera_joint" type="fixed">
-        <origin xyz="0 0 0" rpy="0 0 0"/>
+        <origin xyz="0 0 -0.01" rpy="0 1.05 0"/>
         <parent link="depth_camera_link"/>
         <child link="depth_camera_optical_link"/>
@@ -43,7 +43,12 @@
                 </image>
                 <clip>
-                    <near>0.5</near>
-                    <far>3.0</far>
+                    <near>0.02</near>
+                    <far>300</far>
                 </clip>
+                <noise>
+                    <type>gaussian</type>
+                    <mean>0.0</mean>
+                    <stddev>0.007</stddev>
+                </noise>
             </camera>
             <plugin name="combined_camera_controller" filename="libgazebo_ros_openni_kinect.so">

Commit message: Improve resolution

File: hector_quadrotor_description/urdf/quadrotor_plus.urdf.xacro (robot description, xacro)
@@ -8,6 +8,6 @@
     <!-- Forward facing camera -->
     <xacro:include filename="$(find hector_sensors_description)/urdf/generic_camera_plus.urdf.xacro" />
-    <xacro:generic_camera name="front_cam" parent="camera_link" ros_topic="camera/image" cam_info_topic="camera/camera_info" update_rate="10" res_x="1280" res_y="960" image_format="R8G8B8" hfov="90">
-      <origin xyz="0.0 0.0 0.0" rpy="0 0.5890 0"/>  <!-- PI / 4 = 0.78539 = 45deg -->
+    <xacro:generic_camera name="front_cam" parent="camera_link" ros_topic="camera/image" cam_info_topic="camera/camera_info" update_rate="10" res_x="1920" res_y="1440" image_format="R8G8B8" hfov="90">
+      <origin xyz="0.0 0.0 0.0" rpy="0 0.3490 0"/>  <!-- PI / 4 = 0.78539 = 45deg -->
     </xacro:generic_camera>
     <joint name="depth_camera_joint" type="fixed">
